Commit message: fix-urdf

File: kinova_description/urdf/j2n6s300_standalone.xacro (robot description, xacro)
@@ -17,8 +17,8 @@
   <link name="root"/>
   <!-- for gazebo -->
-  <link name="world"/>
+  <link name="base_link"/>
   <joint name="connect_root_and_world" type="fixed">
     <child link="root" />
-    <parent link="world" />
+    <parent link="base_link" />
     <origin xyz="0 0 0" rpy="0 0 0" />
   </joint>

Commit message: fix-urdf

File: kinova_description/urdf/j2n6s300_standalone.xacro (robot description, xacro)
@@ -14,14 +14,14 @@
     xmlns:physics="http://playerstage.sourceforge.net/gazebo/xmlschema/#physics"
 	xmlns:xacro="http://www.ros.org/wiki/xacro" name="j2n6s300">
-  <xacro:include filename="$(find kinova_description)/urdf/j2n6s300.xacro"/>
-  <link name="root"/>
+  <xacro:include filename="$(find mobiman_simulation)/urdf/jackal_jaco.xacro"/>
+  <!-- <link name="root"/> -->
   <!-- for gazebo -->
-  <link name="base_link"/>
-  <joint name="connect_root_and_world" type="fixed">
-    <child link="root" />
-    <parent link="base_link" />
-    <origin xyz="0 0 0" rpy="0 0 0" />
-  </joint>
-  <xacro:property name="robot_root" value="root" />
-  <xacro:j2n6s300  base_parent="${robot_root}"/>
+  <!-- <link name="base_link"/> -->
+  <!-- <joint name="connect_root_and_world" type="fixed"> -->
+    <!-- <child link="root" /> -->
+    <!-- <parent link="base_link" /> -->
+    <!-- <origin xyz="0 0 0" rpy="0 0 0" />     -->
+  <!-- </joint>  -->
+  <!-- <xacro:property name="robot_root" value="root" /> -->
+  <!-- <xacro:j2n6s300  base_parent="${robot_root}"/> -->
 </robot>

Commit message: fix-urdf

File: kinova_description/urdf/j2n6s300_standalone.xacro (robot description, xacro)
@@ -2,24 +2,24 @@
 <!-- j2n6s300 refers to jaco v2 6DOF non-spherical 3fingers -->
 <robot xmlns:xi="http://www.w3.org/2001/XInclude"
-	xmlns:gazebo="http://playerstage.sourceforge.net/gazebo/xmlschema/#gz"
+        xmlns:gazebo="http://playerstage.sourceforge.net/gazebo/xmlschema/#gz"
     xmlns:model="http://playerstage.sourceforge.net/gazebo/xmlschema/#model"
-	xmlns:sensor="http://playerstage.sourceforge.net/gazebo/xmlschema/#sensor"
-	xmlns:body="http://playerstage.sourceforge.net/gazebo/xmlschema/#body"
+        xmlns:sensor="http://playerstage.sourceforge.net/gazebo/xmlschema/#sensor"
+        xmlns:body="http://playerstage.sourceforge.net/gazebo/xmlschema/#body"
     xmlns:geom="http://playerstage.sourceforge.net/gazebo/xmlschema/#geom"
     xmlns:joint="http://playerstage.sourceforge.net/gazebo/xmlschema/#joint"
-	xmlns:controller="http://playerstage.sourceforge.net/gazebo/xmlschema/#controller"
-	xmlns:interface="http://playerstage.sourceforge.net/gazebo/xmlschema/#interface"
-	xmlns:rendering="http://playerstage.sourceforge.net/gazebo/xmlschema/#rendering"
+        xmlns:controller="http://playerstage.sourceforge.net/gazebo/xmlschema/#controller"
+        xmlns:interface="http://playerstage.sourceforge.net/gazebo/xmlschema/#interface"
+        xmlns:rendering="http://playerstage.sourceforge.net/gazebo/xmlschema/#rendering"
     xmlns:renderable="http://playerstage.sourceforge.net/gazebo/xmlschema/#renderable"
     xmlns:physics="http://playerstage.sourceforge.net/gazebo/xmlschema/#physics"
-	xmlns:xacro="http://www.ros.org/wiki/xacro" name="j2n6s300">
+        xmlns:xacro="http://www.ros.org/wiki/xacro" name="j2n6s300">
   <xacro:include filename="$(find kinova_description)/urdf/j2n6s300.xacro"/>
   <link name="root"/>
   <!-- for gazebo -->
-  <link name="world"/>
+  <link name="base_link"/>
   <joint name="connect_root_and_world" type="fixed">
     <child link="root" />
-    <parent link="world" />
-    <origin xyz="0 0 0" rpy="0 0 0" />
+    <parent link="base_link" />
+    <origin xyz="0 0 0.22" rpy="0 0 0" />
   </joint>
   <xacro:property name="robot_root" value="root" />

Commit message: fix-urdf

File: kinova_description/urdf/j2n6s300_standalone.xacro (robot description, xacro)
@@ -14,8 +14,7 @@
     xmlns:physics="http://playerstage.sourceforge.net/gazebo/xmlschema/#physics"
         xmlns:xacro="http://www.ros.org/wiki/xacro" name="j2n6s300">
-  <xacro:include filename="$(find mobiman_simulation)/urdf/jackal_jaco.xacro"/>
-  <!-- <link name="root"/> -->
+  <xacro:include filename="$(find kinova_description)/urdf/j2n6s300.xacro"/>
+  <link name="root"/>
   <!-- for gazebo -->
-<<<<<<< HEAD
   <link name="base_link"/>
   <joint name="connect_root_and_world" type="fixed">
@@ -24,13 +23,5 @@
     <origin xyz="0 0 0.22" rpy="0 0 0" />
   </joint>
-=======
-  <!-- <link name="base_link"/> -->
-  <!-- <joint name="connect_root_and_world" type="fixed"> -->
-    <!-- <child link="root" /> -->
-    <!-- <parent link="base_link" /> -->
-    <!-- <origin xyz="0 0 0" rpy="0 0 0" />     -->
-  <!-- </joint>  -->
->>>>>>> 187381230519d47d9b0debff55fc5746b4b92243
-  <!-- <xacro:property name="robot_root" value="root" /> -->
-  <!-- <xacro:j2n6s300  base_parent="${robot_root}"/> -->
+  <xacro:property name="robot_root" value="root" />
+  <xacro:j2n6s300  base_parent="${robot_root}"/>
 </robot>
