Commit message: Updated j2n6s300.xacro: updated all arm joints as revolute. Updated kinova_common.xacro: updated friction of arm joints to 0.1 (def:0.0).

File: kinova_description/urdf/j2n6s300.xacro (robot description, xacro)
@@ -44,5 +44,5 @@
     <xacro:property name="joint_base_origin_rpy" value="0 0 0" />
     <xacro:property name="joint_1" value="joint_1" />
-    <xacro:property name="joint_1_type" value="continuous" />
+    <xacro:property name="joint_1_type" value="revolute" />
     <xacro:property name="joint_1_axis_xyz" value="0 0 1" />
     <xacro:property name="joint_1_origin_xyz" value="0 0 0.15675" />
@@ -71,5 +71,5 @@
     <xacro:property name="joint_3_torque_limit" value="40" />
     <xacro:property name="joint_4" value="joint_4" />
-    <xacro:property name="joint_4_type" value="continuous" />
+    <xacro:property name="joint_4_type" value="revolute" />
     <xacro:property name="joint_4_axis_xyz" value="0 0 1" />
     <xacro:property name="joint_4_origin_xyz" value="0 0.2073 -0.0114" />
@@ -80,5 +80,5 @@
     <xacro:property name="joint_4_torque_limit" value="20" />
     <xacro:property name="joint_5" value="joint_5" />
-    <xacro:property name="joint_5_type" value="continuous" />
+    <xacro:property name="joint_5_type" value="revolute" />
     <xacro:property name="joint_5_axis_xyz" value="0 0 1" />
     <xacro:property name="joint_5_origin_xyz" value="0 -0.03703 -0.06414" />
@@ -89,5 +89,5 @@
     <xacro:property name="joint_5_torque_limit" value="20" />
     <xacro:property name="joint_6" value="joint_6" />
-    <xacro:property name="joint_6_type" value="continuous" />
+    <xacro:property name="joint_6_type" value="revolute" />
     <xacro:property name="joint_6_axis_xyz" value="0 0 1" />
     <xacro:property name="joint_6_origin_xyz" value="0 -0.03703 -0.06414" />

File: kinova_description/urdf/kinova_common.xacro (robot description, xacro)
@@ -85,5 +85,5 @@
         </xacro:if>
         <origin xyz="${joint_origin_xyz}" rpy="${joint_origin_rpy}"/>
-        <dynamics damping="0.0" friction="0.0"/>
+        <dynamics damping="0.0" friction="0.1"/>
      </joint>
    <xacro:unless value="${fixed}">

Commit message: Updated j2n6s300.xacro: limits of (continous-by-default but changed to revolute previously) joints 1,4,5,6 are increased to +-200pi.

File: kinova_description/urdf/j2n6s300.xacro (robot description, xacro)
@@ -48,6 +48,6 @@
     <xacro:property name="joint_1_origin_xyz" value="0 0 0.15675" />
     <xacro:property name="joint_1_origin_rpy" value="0 ${J_PI} 0" />
-    <xacro:property name="joint_1_lower_limit" value="${-2*J_PI}" />
-    <xacro:property name="joint_1_upper_limit" value="${2*J_PI}" />
+    <xacro:property name="joint_1_lower_limit" value="${-200*J_PI}" />
+    <xacro:property name="joint_1_upper_limit" value="${200*J_PI}" />
     <xacro:property name="joint_1_velocity_limit" value="${36*J_PI/180}" />
     <xacro:property name="joint_1_torque_limit" value="40" />
@@ -75,6 +75,6 @@
     <xacro:property name="joint_4_origin_xyz" value="0 0.2073 -0.0114" />
     <xacro:property name="joint_4_origin_rpy" value="-${J_PI/2} 0 ${J_PI}" />
-    <xacro:property name="joint_4_lower_limit" value="${-2*J_PI}" />
-    <xacro:property name="joint_4_upper_limit" value="${2*J_PI}" />
+    <xacro:property name="joint_4_lower_limit" value="${-200*J_PI}" />
+    <xacro:property name="joint_4_upper_limit" value="${200*J_PI}" />
     <xacro:property name="joint_4_velocity_limit" value="${48*J_PI/180}" />
     <xacro:property name="joint_4_torque_limit" value="20" />
@@ -84,6 +84,6 @@
     <xacro:property name="joint_5_origin_xyz" value="0 -0.03703 -0.06414" />
     <xacro:property name="joint_5_origin_rpy" value="${J_PI/3} 0 ${J_PI}" />
-    <xacro:property name="joint_5_lower_limit" value="${-2*J_PI}" />
-    <xacro:property name="joint_5_upper_limit" value="${2*J_PI}" />
+    <xacro:property name="joint_5_lower_limit" value="${-200*J_PI}" />
+    <xacro:property name="joint_5_upper_limit" value="${200*J_PI}" />
     <xacro:property name="joint_5_velocity_limit" value="${48*J_PI/180}" />
     <xacro:property name="joint_5_torque_limit" value="20" />
@@ -95,6 +95,6 @@
     <!-- If gripper inverted, use this line instead -->
     <!-- <xacro:property name="joint_6_origin_rpy" value="$${-J_PI/3} 0 0" /> -->
-    <xacro:property name="joint_6_lower_limit" value="${-2*J_PI}" />
-    <xacro:property name="joint_6_upper_limit" value="${2*J_PI}" />
+    <xacro:property name="joint_6_lower_limit" value="${-200*J_PI}" />
+    <xacro:property name="joint_6_upper_limit" value="${200*J_PI}" />
     <xacro:property name="joint_6_velocity_limit" value="${48*J_PI/180}" />
     <xacro:property name="joint_6_torque_limit" value="20" />

Commit message: fixed-urdf

File: kinova_description/urdf/j2n6s300.xacro (robot description, xacro)
@@ -46,5 +46,5 @@
     <xacro:property name="joint_1_type" value="revolute" />
     <xacro:property name="joint_1_axis_xyz" value="0 0 1" />
-    <xacro:property name="joint_1_origin_xyz" value="0 0 0.15675" />
+    <xacro:property name="joint_1_origin_xyz" value="0 0 0.16075" />
     <xacro:property name="joint_1_origin_rpy" value="0 ${J_PI} 0" />
     <xacro:property name="joint_1_lower_limit" value="${-200*J_PI}" />
@@ -122,5 +122,5 @@
         <xacro:kinova_virtual_link link_name="${prefix}_end_effector"/>
         <xacro:kinova_virtual_joint joint_name="${prefix}_joint_end_effector" type="${joint_end_effector_type}" parent="${prefix}_link_6" child="${prefix}_end_effector" joint_axis_xyz="${joint_end_effector_axis_xyz}" joint_origin_xyz="${joint_end_effector_origin_xyz}" joint_origin_rpy="${joint_end_effector_origin_rpy}" joint_lower_limit="0" joint_upper_limit="0"/>
-    <xacro:kinova_3fingers link_hand="${prefix}_link_6" prefix="${prefix}_"/>
+    <!-- <xacro:kinova_3fingers link_hand="${prefix}_link_6" prefix="${prefix}_"/> -->
     </xacro:macro>
 </root>

Commit message: add-more-spacing

File: kinova_description/urdf/j2n6s300.xacro (robot description, xacro)
@@ -46,5 +46,5 @@
     <xacro:property name="joint_1_type" value="revolute" />
     <xacro:property name="joint_1_axis_xyz" value="0 0 1" />
-    <xacro:property name="joint_1_origin_xyz" value="0 0 0.16075" />
+    <xacro:property name="joint_1_origin_xyz" value="0 0 0.16575" />
     <xacro:property name="joint_1_origin_rpy" value="0 ${J_PI} 0" />
     <xacro:property name="joint_1_lower_limit" value="${-200*J_PI}" />

Commit message: Updated j2n6s300.xacro: increased joint_1_origin_xyz to avoid spawning(collision) issues in gazebo.

File: kinova_description/urdf/j2n6s300.xacro (robot description, xacro)
@@ -46,5 +46,5 @@
     <xacro:property name="joint_1_type" value="revolute" />
     <xacro:property name="joint_1_axis_xyz" value="0 0 1" />
-    <xacro:property name="joint_1_origin_xyz" value="0 0 0.16575" />
+    <xacro:property name="joint_1_origin_xyz" value="0 0 0.16975" />
     <xacro:property name="joint_1_origin_rpy" value="0 ${J_PI} 0" />
     <xacro:property name="joint_1_lower_limit" value="${-200*J_PI}" />

Commit message: reset-urdf

File: kinova_description/urdf/j2n6s300.xacro (robot description, xacro)
@@ -46,5 +46,5 @@
     <xacro:property name="joint_1_type" value="revolute" />
     <xacro:property name="joint_1_axis_xyz" value="0 0 1" />
-    <xacro:property name="joint_1_origin_xyz" value="0 0 0.16575" />
+    <xacro:property name="joint_1_origin_xyz" value="0 0 0.15675" />
     <xacro:property name="joint_1_origin_rpy" value="0 ${J_PI} 0" />
     <xacro:property name="joint_1_lower_limit" value="${-200*J_PI}" />
